Commit message: add tests, collision and inertial support

File: tests/model_generated/hexapod_gene.urdf (robot description, URDF)
Before this commit: robot Hopper, 35 links, 34 joints
Joints:
- joint left_front_coxa_joint: axis 0.0 0.0 1.0 -> 0.00000 0.00000 1.00000; limit lower=-3.142 upper=3.142 effort=1000.000 velocity=1.000 -> lower=-3.14159 upper=3.14159 effort=1000.00000 velocity=1.00000
- joint left_front_femur_joint: axis 0.0 0.0 1.0 -> 0.00000 0.00000 1.00000; limit lower=-3.142 upper=3.142 effort=1000.000 velocity=1.000 -> lower=-3.14159 upper=3.14159 effort=1000.00000 velocity=1.00000
- joint left_front_tibia_joint: axis 0.0 0.0 -1.0 -> 0.00000 0.00000 -1.00000; limit lower=-3.142 upper=3.142 effort=1000.000 velocity=1.000 -> lower=-3.14159 upper=3.14159 effort=1000.00000 velocity=1.00000
- joint left_middle_coxa_joint: axis 0.0 0.0 1.0 -> 0.00000 0.00000 1.00000; limit lower=-3.142 upper=3.142 effort=1000.000 velocity=1.000 -> lower=-3.14159 upper=3.14159 effort=1000.00000 velocity=1.00000
- joint left_middle_femur_joint: axis 0.0 0.0 1.0 -> 0.00000 0.00000 1.00000; limit lower=-3.142 upper=3.142 effort=1000.000 velocity=1.000 -> lower=-3.14159 upper=3.14159 effort=1000.00000 velocity=1.00000
- joint left_middle_tibia_joint: axis 0.0 0.0 -1.0 -> 0.00000 0.00000 -1.00000; limit lower=-3.142 upper=3.142 effort=1000.000 velocity=1.000 -> lower=-3.14159 upper=3.14159 effort=1000.00000 velocity=1.00000
- joint left_rear_coxa_joint: axis 0.0 0.0 1.0 -> 0.00000 0.00000 1.00000; limit lower=-3.142 upper=3.142 effort=1000.000 velocity=1.000 -> lower=-3.14159 upper=3.14159 effort=1000.00000 velocity=1.00000
- joint left_rear_femur_joint: axis 0.0 0.0 1.0 -> 0.00000 0.00000 1.00000; limit lower=-3.142 upper=3.142 effort=1000.000 velocity=1.000 -> lower=-3.14159 upper=3.14159 effort=1000.00000 velocity=1.00000
- joint left_rear_tibia_joint: axis 0.0 0.0 -1.0 -> 0.00000 0.00000 -1.00000; limit lower=-3.142 upper=3.142 effort=1000.000 velocity=1.000 -> lower=-3.14159 upper=3.14159 effort=1000.00000 velocity=1.00000
- joint right_front_coxa_joint: axis 0.0 0.0 1.0 -> 0.00000 0.00000 1.00000; limit lower=-3.142 upper=3.142 effort=1000.000 velocity=1.000 -> lower=-3.14159 upper=3.14159 effort=1000.00000 velocity=1.00000
- joint right_front_femur_joint: axis 0.0 0.0 -1.0 -> 0.00000 0.00000 -1.00000; limit lower=-3.142 upper=3.142 effort=1000.000 velocity=1.000 -> lower=-3.14159 upper=3.14159 effort=1000.00000 velocity=1.00000
- joint right_front_tibia_joint: axis 0.0 0.0 1.0 -> 0.00000 0.00000 1.00000; limit lower=-3.142 upper=3.142 effort=1000.000 velocity=1.000 -> lower=-3.14159 upper=3.14159 effort=1000.00000 velocity=1.00000
- joint right_middle_coxa_joint: axis 0.0 0.0 1.0 -> 0.00000 0.00000 1.00000; limit lower=-3.142 upper=3.142 effort=1000.000 velocity=1.000 -> lower=-3.14159 upper=3.14159 effort=1000.00000 velocity=1.00000
- joint right_middle_femur_joint: axis 0.0 0.0 -1.0 -> 0.00000 0.00000 -1.00000; limit lower=-3.142 upper=3.142 effort=1000.000 velocity=1.000 -> lower=-3.14159 upper=3.14159 effort=1000.00000 velocity=1.00000
- joint right_middle_tibia_joint: axis 0.0 0.0 1.0 -> 0.00000 0.00000 1.00000; limit lower=-3.142 upper=3.142 effort=1000.000 velocity=1.000 -> lower=-3.14159 upper=3.14159 effort=1000.00000 velocity=1.00000
- joint right_rear_coxa_joint: axis 0.0 0.0 1.0 -> 0.00000 0.00000 1.00000; limit lower=-3.142 upper=3.142 effort=1000.000 velocity=1.000 -> lower=-3.14159 upper=3.14159 effort=1000.00000 velocity=1.00000
- joint right_rear_femur_joint: axis 0.0 0.0 -1.0 -> 0.00000 0.00000 -1.00000; limit lower=-3.142 upper=3.142 effort=1000.000 velocity=1.000 -> lower=-3.14159 upper=3.14159 effort=1000.00000 velocity=1.00000
- joint right_rear_tibia_joint: axis 0.0 0.0 1.0 -> 0.00000 0.00000 1.00000; limit lower=-3.142 upper=3.142 effort=1000.000 velocity=1.000 -> lower=-3.14159 upper=3.14159 effort=1000.00000 velocity=1.00000
