Commit message: add jenkinsfile and change formatting of numbers in urdf file

File: tests/model_generated/robot_with_geometry_form.urdf (robot description, URDF)
Before this commit: robot test_robot, 2 links, 1 joints
Links:
- link link1: mass 10.0 -> 10; geometry collision box size=3 2 2; visual box size=3 2 2
- link link2: mass 10.0 -> 10

File: tests/model_generated/robot_with_link_only.urdf (robot description, URDF)
Before this commit: robot test_robot, 4 links, 0 joints
Links:
- link link1: mass 1 -> None
- link link2: mass 1 -> None
- link link3: mass 1 -> None
- link link4: mass 1 -> None

File: tests/model_generated/robot_with_one_fixed_joint.urdf (robot description, URDF)
Before this commit: robot test_robot, 4 links, 1 joints
Links:
- link link1: mass 1 -> None
- link link2: mass 1 -> None
- link link3: mass 1 -> None
- link link4: mass 1 -> None

File: tests/model_generated/robot_with_one_revolute_joint.urdf (robot description, URDF)
Before this commit: robot test_robot, 4 links, 1 joints
Links:
- link link1: mass 1 -> None
- link link2: mass 1 -> None
- link link3: mass 1 -> None
- link link4: mass 1 -> None
Joints:
- joint fixed_joint: axis 0.00000 1.00000 0.00000 -> 0 1 0; limit lower=-3.14159 upper=3.14159 effort=1000.00000 velocity=1.00000 -> lower=-3.14159 upper=3.14159 effort=1000 velocity=1

File: tests/reference_model/robot_with_geometry_form.urdf (robot description, URDF)
Before this commit: robot test_robot, 2 links, 1 joints
Links:
- link link1: mass 10.0 -> 10; geometry collision box size=3 2 2; visual box size=3 2 2
- link link2: mass 10.0 -> 10

File: tests/reference_model/robot_with_one_revolute_joint.urdf (robot description, URDF)
Before this commit: robot test_robot, 4 links, 1 joints
Joints:
- joint fixed_joint: axis 0.00000 1.00000 0.00000 -> 0 1 0; limit lower=-3.14159 upper=3.14159 effort=1000.00000 velocity=1.00000 -> lower=-3.14159 upper=3.14159 effort=1000 velocity=1

Commit message: change completely structure to ease designer development

File: tests/model_generated/robot_with_geometry_form.urdf (robot description, URDF)
Before this commit: robot test_robot, 2 links, 1 joints
Links:
- removed link link1
- added link base_link, mass 10; collision box size=3 2 2; visual box size=3 2 2
Joints:
- joint fixed_joint: parent link1 -> base_link

File: tests/model_generated/robot_with_link_only.urdf (robot description, URDF)
Before this commit: robot test_robot, 4 links, 0 joints
Links:
- removed link link1
- removed link link2
- removed link link3
- removed link link4
- added link base_link

File: tests/model_generated/robot_with_one_fixed_joint.urdf (robot description, URDF)
Before this commit: robot test_robot, 4 links, 1 joints
Links:
- removed link link3
- removed link link4

File: tests/model_generated/robot_with_one_revolute_joint.urdf (robot description, URDF)
Before this commit: robot test_robot, 4 links, 1 joints
Links:
- removed link link3
- removed link link4

File: tests/reference_model/robot_with_geometry_form.urdf (robot description, URDF)
Before this commit: robot test_robot, 2 links, 1 joints
Links:
- removed link link1
- added link base_link, mass 10; collision box size=3 2 2; visual box size=3 2 2
Joints:
- joint fixed_joint: parent link1 -> base_link

File: tests/reference_model/robot_with_link_only.urdf (robot description, URDF)
Before this commit: robot test_robot, 4 links, 0 joints
Links:
- removed link link1
- removed link link2
- removed link link3
- removed link link4
- added link base_link

File: tests/reference_model/robot_with_one_fixed_joint.urdf (robot description, URDF)
Before this commit: robot test_robot, 4 links, 1 joints
Links:
- removed link link3
- removed link link4

File: tests/reference_model/robot_with_one_revolute_joint.urdf (robot description, URDF)
Before this commit: robot test_robot, 4 links, 1 joints
Links:
- removed link link3
- removed link link4
