Commit message: change dockerfile to work

File: tests/model_generated/rrbot.urdf (robot description, URDF)
Before this commit: robot rrbot, 7 links, 6 joints
Joints:
- joint camera_joint: origin xyz=<simpleurdf.urdf2model.basemodel.Box object at 0x7f82031e0730> 0.0 0.9 rpy=0 0 0 -> xyz=<simpleurdf.urdf2model.basemodel.Box object at 0x7f2973715580> 0.0 0.9 rpy=0 0 0

Commit message: add nested models, add tests and fix bugs

File: tests/model_generated/rrbot.urdf (robot description, URDF)
Before this commit: robot rrbot, 7 links, 6 joints
Joints:
- joint camera_joint: origin xyz=<simpleurdf.urdf2model.basemodel.Box object at 0x7f2973715580> 0.0 0.9 rpy=0 0 0 -> xyz=0.05 0 0.9 rpy=0 0 0
