Commit message: modify box  to corresponds to reality

File: tests/model_generated/model_in_model.urdf (robot description, URDF)
Before this commit: robot test_robot, 2 links, 1 joints
Links:
- link base_link: geometry collision box size=2 2 3; visual box size=2 2 3

File: tests/model_generated/robot_with_geometry_form.urdf (robot description, URDF)
Before this commit: robot test_robot, 2 links, 1 joints
Links:
- link base_link: geometry collision box size=2 2 3; visual box size=2 2 3
